File: Neo6502.kicad_sch (KiCad schematic)
At the start: 65 parts, among them J1 DE15_Receptacle_HighDensity, J2 USB_B, SW1 SW_Push, SW10 SW_Push, SW11 SW_DIP_x02, SW2 SW_Push, SW3 SW_Push, SW4 SW_Push, SW5 SW_Push, SW6 SW_Push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

Commit message: Add files via upload
Connections:
- net SIXTEENTH: now reaches U7.11 (Q3)
- no-connect marks 22 -> 21
Other:
- note added: "DS should have been grounded!"
- note added: "Needs to be SIXTEENTH instead!"
- note added: "Outputs should be switched!"
- note removed: "DS should have been grounded."
Changed lines of the file:
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@@
   (no_connect (at 46.99 387.35))
   (no_connect (at 99.06 157.48))
-  (no_connect (at 134.62 213.36))
   (no_connect (at 62.23 377.19))
   (no_connect (at 99.06 149.86))
@@
     (effects (font (size 1.27 1.27)) (justify left bottom))
   )
+  (text "Needs to be SIXTEENTH instead!" (at 153.67 361.95 90)
+    (effects (font (size 1.27 1.27)) (justify left bottom))
+  )
   (text "79.4ns" (at 12.7 431.8 0)
     (effects (font (size 1.27 1.27)) (justify left bottom))
@@
     (effects (font (size 1.27 1.27)) (justify left bottom))
   )
-  (text "DS should have been grounded." (at 207.01 191.77 90)
+  (text "DS should have been grounded!" (at 207.01 191.77 90)
+    (effects (font (size 1.27 1.27)) (justify left bottom))
+  )
+  (text "Outputs should be switched!" (at 238.76 82.55 90)
     (effects (font (size 1.27 1.27)) (justify left bottom))
   )
@@
     )
   )
+  (global_label "SIXTEENTH" (shape input) (at 134.62 213.36 0) (fields_autoplaced)
+    (effects (font (size 1.27 1.27)) (justify left))
+    (property "Intersheetrefs" "${INTERSHEET_REFS}" (at 147.5232 213.36 0)
+      (effects (font (size 1.27 1.27)) (justify left) hide)
+    )
+  )
